File: Projects/Pippino_board_v2/pippino_board/adc_block.kicad_sch (KiCad schematic)
At the start: 9 parts, among them U7 ADS1115IDGS

Commit message: added pippino board v2
Parts:
- renumbered C5 to C6, C6 to C7, R11 to R16, R12 to R17, R13 to R18, R14 to R19, U7 to U4
Changed lines of the file:
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@@
   (symbol (lib_id "power:GND") (at 152.4 96.52 0) (unit 1)
     (in_bom yes) (on_board yes) (fields_autoplaced)
-    (property "Reference" "#PWR039" (id 0) (at 152.4 102.87 0)
+    (property "Reference" "#PWR038" (id 0) (at 152.4 102.87 0)
       (effects (font (size 1.27 1.27)) hide)
     )
@@
   (symbol (lib_id "Device:R") (at 175.26 92.71 0) (unit 1)
     (in_bom yes) (on_board yes) (fields_autoplaced)
-    (property "Reference" "R12" (id 0) (at 177.8 91.4399 0)
+    (property "Reference" "R17" (id 0) (at 177.8 91.4399 0)
       (effects (font (size 1.27 1.27)) (justify left))
     )
@@
   (symbol (lib_id "power:GND") (at 91.44 102.87 0) (unit 1)
     (in_bom yes) (on_board yes) (fields_autoplaced)
-    (property "Reference" "#PWR038" (id 0) (at 91.44 109.22 0)
+    (property "Reference" "#PWR037" (id 0) (at 91.44 109.22 0)
       (effects (font (size 1.27 1.27)) hide)
     )
@@
   (symbol (lib_id "Analog_ADC:ADS1115IDGS") (at 152.4 81.28 0) (unit 1)
     (in_bom yes) (on_board yes) (fields_autoplaced)
-    (property "Reference" "U7" (id 0) (at 154.4194 66.04 0)
+    (property "Reference" "U4" (id 0) (at 154.4194 66.04 0)
       (effects (font (size 1.27 1.27)) (justify left))
     )
@@
   (symbol (lib_id "power:GND") (at 161.29 66.04 0) (unit 1)
     (in_bom yes) (on_board yes) (fields_autoplaced)
-    (property "Reference" "#PWR040" (id 0) (at 161.29 72.39 0)
+    (property "Reference" "#PWR039" (id 0) (at 161.29 72.39 0)
       (effects (font (size 1.27 1.27)) hide)
     )
@@
   (symbol (lib_id "Device:R") (at 180.34 68.58 0) (unit 1)
     (in_bom yes) (on_board yes) (fields_autoplaced)
-    (property "Reference" "R13" (id 0) (at 182.88 67.3099 0)
+    (property "Reference" "R18" (id 0) (at 182.88 67.3099 0)
       (effects (font (size 1.27 1.27)) (justify left))
     )
@@
   (symbol (lib_id "Device:R") (at 168.91 68.58 0) (unit 1)
     (in_bom yes) (on_board yes) (fields_autoplaced)
-    (property "Reference" "R11" (id 0) (at 171.45 67.3099 0)
+    (property "Reference" "R16" (id 0) (at 171.45 67.3099 0)
       (effects (font (size 1.27 1.27)) (justify left))
     )
@@
   (symbol (lib_id "Device:C") (at 161.29 62.23 0) (unit 1)
     (in_bom yes) (on_board yes) (fields_autoplaced)
-    (property "Reference" "C6" (id 0) (at 165.1 60.9599 0)
+    (property "Reference" "C7" (id 0) (at 165.1 60.9599 0)
       (effects (font (size 1.27 1.27)) (justify left))
     )
@@
   (symbol (lib_id "power:GND") (at 175.26 99.06 0) (unit 1)
     (in_bom yes) (on_board yes) (fields_autoplaced)
-    (property "Reference" "#PWR041" (id 0) (at 175.26 105.41 0)
+    (property "Reference" "#PWR040" (id 0) (at 175.26 105.41 0)
       (effects (font (size 1.27 1.27)) hide)
     )
@@
   (symbol (lib_id "Device:C") (at 91.44 81.28 0) (unit 1)
     (in_bom yes) (on_board yes) (fields_autoplaced)
-    (property "Reference" "C5" (id 0) (at 95.25 80.0099 0)
+    (property "Reference" "C6" (id 0) (at 95.25 80.0099 0)
       (effects (font (size 1.27 1.27)) (justify left))
     )
@@
   (symbol (lib_id "Device:R") (at 190.5 68.58 0) (unit 1)
     (in_bom yes) (on_board yes) (fields_autoplaced)
-    (property "Reference" "R14" (id 0) (at 193.04 67.3099 0)
-      (effects (font (size 1.27 1.27)) (justify left))
-    )
+    (property "Reference" "R19" (id 0) (at 193.04 67.3099 0)
+      (effects (font (size 1.27 1.27)) (justify left))
+    )
