File: Projects/Pippino_board_v2/pippino_board/dc_motor_driver.kicad_sch (KiCad schematic)
At the start: 3 parts, among them U5 DRV8871DDA

Commit message: added pippino board v2
Parts:
- renumbered C2 to C3, R5 to R8, U5 to U2
Changed lines of the file:
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@@
     (effects (font (size 1.27 1.27)) (justify right))
   )
-  (symbol (lib_id "Device:R") (at 133.35 78.74 0)
+  (symbol (lib_id "Device:R") (at 133.35 78.74 0) (unit 1)
     (in_bom yes) (on_board yes) (fields_autoplaced)
-    (property "Reference" "R5" (id 0) (at 135.89 77.4699 0)
+    (property "Reference" "R8" (id 0) (at 135.89 77.4699 0)
       (effects (font (size 1.27 1.27)) (justify left))
     )
@@
     (pin "2")
   )
-  (symbol (lib_id "Device:C") (at 168.91 63.5 0)
+  (symbol (lib_id "Device:C") (at 168.91 63.5 0) (unit 1)
     (in_bom yes) (on_board yes) (fields_autoplaced)
-    (property "Reference" "C2" (id 0) (at 172.72 62.2299 0)
+    (property "Reference" "C3" (id 0) (at 172.72 62.2299 0)
       (effects (font (size 1.27 1.27)) (justify left))
     )
@@
     (pin "2")
   )
-  (symbol (lib_id "Driver_Motor:DRV8871DDA") (at 118.11 69.85 0)
+  (symbol (lib_id "Driver_Motor:DRV8871DDA") (at 118.11 69.85 0) (unit 1)
     (in_bom yes) (on_board yes) (fields_autoplaced)
-    (property "Reference" "U5" (id 0) (at 120.1294 59.69 0)
+    (property "Reference" "U2" (id 0) (at 120.1294 59.69 0)
       (effects (font (size 1.27 1.27)) (justify left))
     )
@@
     (pin "9")
   )
-  (symbol (lib_id "power:GND") (at 118.11 87.63 0)
+  (symbol (lib_id "power:GND") (at 118.11 87.63 0) (unit 1)
     (in_bom yes) (on_board yes) (fields_autoplaced)
     (property "Reference" "#PWR031" (id 0) (at 118.11 93.98 0)
