File: Projects/Pippino_board_v2/pippino_board/pippino_board.kicad_pcb (KiCad board)
At the start: 2 copper layers, 97 x 57 mm, 56 parts, among them J1 Conn_02x01, J10 Conn_01x06, J11 Conn_01x02, J2 Conn_02x02_Counter_Clockwise, J3 Conn_02x07_Odd_Even, J4 Conn_01x04, J5 Conn_01x06, J6 Conn_01x04, J7 Conn_01x04, J8 Conn_01x04, J9 Conn_01x06, Q1 2N3904, Q2 NDP6020P, Q3 NDP6020P, SW1 SW_Push, U1 ESP32-DevKitC, U2 Mini360, U3 E18-MS1-PCB, U4 DRV8871DDA, U5 DRV8871DDA, U6 CKCS_BK03, U7 ADS1115IDGS

Commit message: added pippino board v2
Parts:
- removed MH1, MH2, MH4: MountingHole_3mm, MountingHole:MountingHole_3mm
- added C10: 10p, Capacitor_SMD:C_0805_2012Metric, F.Cu at (145.1, 114.9)
- added C11: 22u, Capacitor_SMD:C_0805_2012Metric, F.Cu at (145.1, 111.9)
- added C12: 10uF, Capacitor_SMD:C_0805_2012Metric, F.Cu at (40.0, 99.3)
- added C13: 1uF, Capacitor_SMD:C_0805_2012Metric, F.Cu at (24.9, 111.0)
- added C14: 1uF, Capacitor_SMD:C_0805_2012Metric, F.Cu at (52.5, 86.6)
- added C15: 10uF, Capacitor_SMD:C_0805_2012Metric, F.Cu at (149.5, 80.0)
- added C16: 1uF, Capacitor_SMD:C_0805_2012Metric, F.Cu at (165.5, 64.7)
- added C17: 100n, Capacitor_SMD:C_0805_2012Metric, F.Cu at (145.1, 80.0)
- added C18: 10uF, Capacitor_SMD:C_0805_2012Metric, F.Cu at (118.1, 117.3)
- added C19: 1u, Capacitor_SMD:C_0805_2012Metric, F.Cu at (112.5, 120.6)
- added C20: 10p, Capacitor_SMD:C_0805_2012Metric, F.Cu at (123.7, 114.0)
- added C21: 22u, Capacitor_SMD:C_0805_2012Metric, F.Cu at (117.0, 120.6)
- added C22: 100n, Capacitor_SMD:C_0805_2012Metric, F.Cu at (132.9, 99.7)
- added D10: ESD9B5.0ST5G, Diode_SMD:D_SOD-923, F.Cu at (46.7, 93.3)
- added D4: LED, LED_SMD:LED_1206_3216Metric, F.Cu at (73.4, 47.4)
- added D5: LED, LED_SMD:LED_1206_3216Metric, F.Cu at (54.0, 66.2)
- added D6: 1N5819, Diode_SMD:D_SMA, F.Cu at (107.5, 70.8)
- added D7: 1N5819, Diode_SMD:D_SMA, F.Cu at (99.1, 77.2)
- added D8: ESD9B5.0ST5G, Diode_SMD:D_SOD-923, F.Cu at (44.0, 93.3)
- added D9: ESD9B5.0ST5G, Diode_SMD:D_SOD-923, F.Cu at (57.3, 82.7)
- added J12: IO, Connector_PinHeader_2.54mm:PinHeader_2x05_P2.54mm_Vertical_SMD, F.Cu at (101.5, 40.8)
- added J13: IO, Connector_PinHeader_2.54mm:PinHeader_2x05_P2.54mm_Vertical_SMD, F.Cu at (101.5, 55.6)
- added J14: USB_B_Micro, Connector_USB:USB_Micro-B_Molex_47346-0001, F.Cu at (37.4, 90.1)
- added L1: 6.8u 2A, Inductor_SMD:L_Bourns_SRN6045TA, F.Cu at (137.2, 91.4)
- added L2: 6.8u 2A, Inductor_SMD:L_Bourns_SRN6045TA, F.Cu at (117.7, 105.3)
- added Q4: L8050_SOT23, Package_TO_SOT_SMD:SOT-23, F.Cu at (50.7, 91.2)
- added R15: 220K, Resistor_SMD:R_1206_3216Metric, F.Cu at (111.5, 74.7)
- added R16: 10k, Resistor_SMD:R_1206_3216Metric, F.Cu at (90.4, 107.8)
- added R17: 10k, Resistor_SMD:R_1206_3216Metric, F.Cu at (90.4, 104.5)
- added R18: 10k, Resistor_SMD:R_1206_3216Metric, F.Cu at (97.3, 99.9)
- added R19: 10k, Resistor_SMD:R_1206_3216Metric, F.Cu at (90.4, 111.1)
- added R20: 560K, Resistor_SMD:R_1206_3216Metric, F.Cu at (160.9, 35.1)
- added R21: 300K, Resistor_SMD:R_1206_3216Metric, F.Cu at (160.9, 38.4)
- added R22: 1M, Resistor_SMD:R_1206_3216Metric, F.Cu at (145.7, 108.8)
- added R23: 560K, Resistor_SMD:R_1206_3216Metric, F.Cu at (122.9, 70.2)
- added R24: 300K, Resistor_SMD:R_1206_3216Metric, F.Cu at (122.9, 73.4)
- added R25: 10k, Resistor_SMD:R_1206_3216Metric, F.Cu at (121.3, 35.1)
- added R26: 10k, Resistor_SMD:R_1206_3216Metric, F.Cu at (126.9, 35.1)
- added R27: 22.1K, Resistor_SMD:R_1206_3216Metric, F.Cu at (35.0, 99.4)
- added R28: 47.5K, Resistor_SMD:R_1206_3216Metric, F.Cu at (35.0, 96.1)
- added R29: 1K, Resistor_SMD:R_1206_3216Metric, F.Cu at (14.3, 111.1)
- added R30: 10K(NC), Resistor_SMD:R_1206_3216Metric, F.Cu at (19.9, 111.1)
- added R31: 10K(NC), Resistor_SMD:R_1206_3216Metric, F.Cu at (45.5, 90.7)
- added R32: 10K, Resistor_SMD:R_1206_3216Metric, F.Cu at (53.1, 83.4)
- added R33: 10K, Resistor_SMD:R_1206_3216Metric, F.Cu at (40.6, 96.1)
- added R34: 720K, Resistor_SMD:R_1206_3216Metric, F.Cu at (113.1, 117.4)
- added R35: 100K, Resistor_SMD:R_1206_3216Metric, F.Cu at (118.7, 114.1)
- added R36: 1M, Resistor_SMD:R_1206_3216Metric, F.Cu at (113.1, 114.1)
- added R37: 1M, Resistor_SMD:R_1206_3216Metric, F.Cu at (127.8, 99.9)
- added SW2: SW_Push, Button_Switch_SMD:SW_SPST_CK_RS282G05A3, F.Cu at (37.6, 84.3)
- added U10: TPS62110, Package_DFN_QFN:HVQFN-16-1EP_3x3mm_P0.5mm_EP1.5x1.5mm, F.Cu at (127.7, 104.2)
- added U8: ESP32-S3-WROOM-1, Espressif:ESP32-S3-WROOM-1, F.Cu at (193.0, 43.2)
- added U9: CKCS_BK03, Pcb_Modules:CKCS-BK03, F.Cu at (228.6, 96.5)
- C1: value 0.1uF -> 10uF
- C2: value 0.1uF -> 470uF; footprint Capacitor_SMD:C_0805_2012Metric -> Capacitor_SMD:CP_Elec_10x10.5
- C3, C4: value 10uF -> 0.1uF
- C5: value 1uF -> 10uF
- C7: value 47uF -> 1uF; footprint Capacitor_SMD:CP_Elec_6.3x5.4 -> Capacitor_SMD:C_0805_2012Metric
- C8: value 100nF -> 10uF
- C9: value 47uF -> 1u; footprint Capacitor_SMD:CP_Elec_6.3x5.4 -> Capacitor_SMD:C_0805_2012Metric
- D2, D3: value 1N5819 -> LED; footprint Diode_SMD:D_SMA -> LED_SMD:LED_1206_3216Metric
- J10: value Conn_01x06 -> Conn_02x03; footprint Connector_JST:JST_PH_B6B-PH-K_1x06_P2.00mm_Vertical -> Connector_PinHeader_2.54mm:PinHeader_2x03_P2.54mm_Vertical_SMD
- J11: value Conn_01x02 -> Conn_02x03; footprint Connector_PinHeader_2.54mm:PinHeader_1x02_P2.54mm_Horizontal -> Connector_PinHeader_2.54mm:PinHeader_2x03_P2.54mm_Vertical_SMD
- J2: value Conn_02x02_Counter_Clockwise -> Conn_02x09_Odd_Even; footprint Connector_Molex:Molex_Micro-Fit_3.0_43045-0400_2x02_P3.00mm_Horizontal -> Connector_PinHeader_2.54mm:PinHeader_2x09_P2.54mm_Vertical_SMD
- J3: value Conn_02x07_Odd_Even -> Conn_01x04; footprint Connector_PinHeader_2.54mm:PinHeader_2x07_P2.54mm_Vertical -> Connector_PinHeader_2.54mm:PinHeader_1x04_P2.54mm_Vertical_SMD_Pin1Left
- J4: value Conn_01x04 -> Conn_01x06; footprint Connector_PinHeader_2.54mm:PinHeader_1x04_P2.54mm_Vertical -> Connector_PinHeader_2.54mm:PinHeader_1x06_P2.54mm_Vertical_SMD_Pin1Left
- J5: value Conn_01x06 -> Conn_02x02_Counter_Clockwise; footprint Connector_PinHeader_2.54mm:PinHeader_1x06_P2.54mm_Vertical -> Connector_Molex:Molex_Micro-Fit_3.0_43045-0400_2x02_P3.00mm_Horizontal
- J6, J7: footprint Connector_PinHeader_2.54mm:PinHeader_1x04_P2.54mm_Vertical -> Connector_PinHeader_2.54mm:PinHeader_1x04_P2.54mm_Vertical_SMD_Pin1Left
- J8: value Conn_01x04 -> Conn_01x06; footprint Connector_PinHeader_2.54mm:PinHeader_1x04_P2.54mm_Vertical -> Connector_JST:JST_PH_B6B-PH-K_1x06_P2.00mm_Vertical
- Q1: footprint Components:2N3904_SOT-23 -> Package_TO_SOT_SMD:SOT-23
- Q2: value NDP6020P -> AO4409; footprint NDP6020P:TO254P470X1016X2019-3P -> Package_SO:SOIC-8_3.9x4.9mm_P1.27mm
- Q3: value NDP6020P -> L8050_SOT23; footprint NDP6020P:TO254P470X1016X2019-3P -> Package_TO_SOT_SMD:SOT-23
- R1, R3, R5: value 18k -> 330
- R10: value 330 -> 220K
- R11, R14: value 10k -> 220
- R12: value 10k -> 100K
- R13: value 10k -> 100k
- R4: value 5.1k -> 330
- R6: value 220k -> 18k
- R7: value 330 -> 5.1k
- R8, R9: value 100k -> 18k
- U1: value ESP32-DevKitC -> E18-MS1-PCB; footprint PCB Modules:ESP32_DevKitC_V4 -> RF_Module:E18-MS1-PCB
- U2: value Mini360 -> DRV8871DDA; footprint PCB Modules:Mini360 -> Package_SO:Texas_HTSOP-8-1EP_3.9x4.9mm_P1.27mm_EP2.95x4.9mm_Mask2.4x3.1mm_ThermalVias
- U3: value E18-MS1-PCB -> DRV8871DDA; footprint RF_Module:E18-MS1-PCB -> Package_SO:Texas_HTSOP-8-1EP_3.9x4.9mm_P1.27mm_EP2.95x4.9mm_Mask2.4x3.1mm_ThermalVias
- U4: value DRV8871DDA -> ADS1115IDGS; footprint Package_SO:Texas_HTSOP-8-1EP_3.9x4.9mm_P1.27mm_EP2.95x4.9mm_Mask2.4x3.1mm_ThermalVias -> Package_SO:TSSOP-10_3x3mm_P0.5mm
- U5: value DRV8871DDA -> TPS62110; footprint Package_SO:Texas_HTSOP-8-1EP_3.9x4.9mm_P1.27mm_EP2.95x4.9mm_Mask2.4x3.1mm_ThermalVias -> Package_DFN_QFN:HVQFN-16-1EP_3x3mm_P0.5mm_EP1.5x1.5mm
- U6: value CKCS_BK03 -> MCP23017; footprint PCB Modules:CKCS-BK03 -> Package_SO:SSOP-28_5.3x10.2mm_P0.65mm
- U7: value ADS1115IDGS -> CP2102N-Axx-xQFN28; footprint Package_SO:TSSOP-10_3x3mm_P0.5mm -> Package_DFN_QFN:QFN-28-1EP_5x5mm_P0.5mm_EP3.35x3.35mm
- moved J4 235.0 mm to (15.5, 67.7), turned to 0 degrees
- moved J7 204.2 mm to (47.2, 71.1), turned to 0 degrees
- moved U7 188.9 mm to (46.7, 85.4), turned to 0 degrees
- moved J11 177.9 mm to (64.4, 38.3), turned to 0 degrees
- moved D1 169.4 mm to (22.3, 75.4), turned to 0 degrees
- moved J8 168.4 mm to (32.1, 61.1), turned to 0 degrees
- moved C2 149.6 mm to (36.1, 71.0), turned to 0 degrees
- moved J10 148.4 mm to (51.5, 59.6), turned to 0 degrees
- moved C6 147.6 mm to (101.0, 103.0), turned to 0 degrees
- moved R4 146.1 mm to (54.0, 72.9)
- moved JP1 144.9 mm to (60.3, 57.8), turned to 0 degrees
- moved R14 142.8 mm to (97.9, 84.4), turned to 0 degrees
- moved R11 140.1 mm to (97.9, 81.2), turned to 0 degrees
- moved FB2 139.6 mm to (96.0, 104.5)
- moved J3 137.7 mm to (74.8, 39.6)
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Connections:
- C1 pad 1: VBATT_GATED -> +3V3
- C2 pad 1: VBATT_GATED -> +BATT
- C4 pad 1: 5V_GATED -> VBATT_GATED
- C5 pad 1: Net-(C5-Pad1) -> VBATT_GATED
- C5 pad 2: Net-(C5-Pad2) -> GND
- C6 pad 1: 3V3_ESP32 -> Net-(C6-Pad1)
- C6 pad 2: GND -> Net-(C6-Pad2)
- C7 pad 1: +3V3 -> 3V3_GATED
- C8 pad 1: +3V3 -> VBATT_GATED
- C9 pad 1: +BATT -> VBATT_GATED
- D1 pad 2: 5V_GATED -> /LED1
- D2 pad 2: Net-(D2-Pad2) -> /LED2
- D3 pad 1: Net-(D2-Pad1) -> Net-(D3-Pad1)
- D3 pad 2: Net-(D3-Pad2) -> /ESPIO19
- FB1 pad 1: 3V3_ESP32 -> 3V3_GATED
- FB1 pad 2: Net-(C5-Pad1) -> Net-(C6-Pad1)
- FB2 pad 1: Net-(C5-Pad2) -> Net-(C6-Pad2)
- J10 pad 1: /M2+ -> GND
- J10 pad 2: GND -> /M1enc1
- J10 pad 3: /M2enc2 -> VBATT_GATED
- J10 pad 4: /M2enc1 -> /M1PWM1
- J10 pad 5: 3V3_ESP32 -> /M1enc2_dir
- J10 pad 6: /M2- -> /M1PWM2_brake
- J11 pad 1: /RXD0 -> GND
- J11 pad 2: /TXD0 -> /M2enc1
- J2 pad 1: GND -> +3V3
- J2 pad 3: 5V_GATED -> /EXT1
- J2 pad 4: VBATT_GATED -> /ESPEN
- J3 pad 2: GND -> /ESPIO11
- J3 pad 3: /EXT1 -> /ESPIO12
- J3 pad 4: /ESPEN -> GND
- J4 pad 2: /ESPIO15 -> /MOSI
- J4 pad 3: /ESPIO4 -> /MISO
- J4 pad 4: GND -> /SPICLK
- J5 pad 1: +3V3 -> GND
- J5 pad 2: /MOSI -> GND
- J5 pad 3: /MISO -> 5V0_GATED
- J5 pad 4: /SPICLK -> VBATT_GATED
- J6 pad 2: /ESPIO16 -> /ESPIO13
- J6 pad 3: /ESPIO17 -> /ESPIO14
- J8 pad 1: +3V3 -> /M1+
- J8 pad 2: /ESPIO39 -> GND
- J8 pad 3: /ESPIO13 -> /M1enc2_dir
- J8 pad 4: GND -> /M1enc1
- J9 pad 1: /M1+ -> /M2+
- J9 pad 3: /M1enc2 -> /M2enc2_dir
- J9 pad 4: /M1enc1 -> /M2enc1
- J9 pad 5: 3V3_ESP32 -> 3V3_GATED
- J9 pad 6: /M1- -> /M2-
- JP1 pad 3: /ESPIO16 -> /ESPIO35
- JP2 pad 3: /E18P17 -> /E18P10
- Q1 pad 2: Net-(D2-Pad1) -> /VBATT_trig_manual
- Q2 pad 1: Net-(Q1-Pad3) -> (no net)
- Q2 pad 2: VBATT_GATED -> (no net)
- Q2 pad 3: +BATT -> (no net)
- Q3 pad 1: Net-(Q1-Pad3) -> Net-(Q3-Pad1)
- Q3 pad 2: VBATT_GATED -> /ESP32_Module/RTS
- Q3 pad 3: +BATT -> /ESPEN
- R1 pad 1: Net-(R1-Pad1) -> Net-(D1-Pad1)
- R10 pad 1: Net-(D3-Pad2) -> /VBATT_trigger
- R10 pad 2: /VBATT_maintain -> GND
- R11 pad 1: 3V3_ESP32 -> /VBATT_trigger
- R11 pad 2: Net-(R11-Pad2) -> Net-(D6-Pad2)
- R12 pad 1: Net-(R12-Pad1) -> +BATT
- R12 pad 2: GND -> Net-(Q1-Pad3)
- R13 pad 1: 3V3_ESP32 -> /VBATT_trig_manual
- R13 pad 2: /SCL -> GND
- R14 pad 1: 3V3_ESP32 -> Net-(D7-Pad2)
- R14 pad 2: /SDA -> /VBATT_maintain
- R2 pad 1: Net-(D1-Pad1) -> Net-(D2-Pad1)
- R3 pad 1: VBATT_GATED -> Net-(D3-Pad1)
- R3 pad 2: /ADC/ADS_IN1 -> GND
- R4 pad 1: /ADC/ADS_IN1 -> Net-(D4-Pad1)
- R5 pad 1: Net-(R5-Pad1) -> Net-(D5-Pad1)
- R6 pad 1: /VBATT_trigger -> VBATT_GATED
- R6 pad 2: GND -> /ADC/ADS_IN1
- R7 pad 1: /VBATT_trigger -> /ADC/ADS_IN1
- R7 pad 2: Net-(D2-Pad2) -> GND
- R8 pad 1: +BATT -> Net-(R8-Pad1)
- R8 pad 2: Net-(Q1-Pad3) -> GND
- R9 pad 1: Net-(D2-Pad1) -> Net-(R9-Pad1)
- SW1 pad 2: /VBATT_trigger -> /VBATT_trig_manual
- U1 pad 1: 3V3_ESP32 -> GND
- U1 pad 10: /M2PWM2 -> /E18P15
- U1 pad 11: /M1PWM1 -> /E18P14
- U1 pad 12: /E18RX -> /RUN_LED
- U1 pad 13: /M1PWM2 -> /NWK_LED
- U1 pad 14: GND -> unconnected-(U1-Pad14)
- U1 pad 15: /ESPIO13 -> /E18P10
- U1 pad 19: 5V_GATED -> unconnected-(U1-Pad19)
- U1 pad 2: /ESPEN -> +3V3
- U1 pad 20: unconnected-(U1-Pad20) -> /E18TX
- U1 pad 21: unconnected-(U1-Pad21) -> /E18RX
- U1 pad 23: /ESPIO15 -> unconnected-(U1-Pad23)
- U1 pad 24: unconnected-(U1-Pad24) -> /E18RST
- U1 pad 3: /E18TX -> /E18DC
- U1 pad 4: /ESPIO39 -> /E18DD
- U1 pad 5: /M2enc2 -> unconnected-(U1-Pad5)
- U1 pad 6: /M2enc1 -> /Batt_Low_Flag
- U1 pad 7: /M1enc2 -> /E18P16
- U1 pad 8: /M1enc1 -> unconnected-(U1-Pad8)
- U1 pad 9: /M2PWM1 -> unconnected-(U1-Pad9)
- U2 pad 2: +BATT -> /M1PWM2_brake
- U2 pad 3: GND -> /M1PWM1
- U2 pad 4: +3V3 -> Net-(R8-Pad1)
- U3 pad 2: +3V3 -> /M2PWM2_brake
- U3 pad 3: /E18DC -> /M2PWM1
- U3 pad 4: /E18DD -> Net-(R9-Pad1)
- U3 pad 5: unconnected-(U3-Pad5) -> VBATT_GATED
- U3 pad 6: /E18P17 -> /M2+
- U3 pad 7: /E18P16 -> GND
- U3 pad 8: unconnected-(U3-Pad8) -> /M2-
- U3 pad 9: unconnected-(U3-Pad9) -> GND
- U4 pad 1: GND -> Net-(R17-Pad1)
- U4 pad 2: /M1PWM2 -> Net-(R16-Pad2)
- U4 pad 3: /M1PWM1 -> GND
- U4 pad 4: Net-(R1-Pad1) -> /ADS0
- U4 pad 5: VBATT_GATED -> /ADC/ADS_IN1
- U4 pad 6: /M1+ -> /ADS2
- U4 pad 7: GND -> /ADS3
- U4 pad 8: /M1- -> 3V3_GATED
- U4 pad 9: GND -> /SDA_INT
- U5 pad 2: /M2PWM2 -> VBATT_GATED
- U5 pad 3: /M2PWM1 -> VBATT_GATED
- U5 pad 4: Net-(R5-Pad1) -> VBATT_GATED
- U5 pad 5: VBATT_GATED -> GND
- U5 pad 6: /M2+ -> unconnected-(U5-Pad6)
- U5 pad 8: /M2- -> VBATT_GATED
- U6 pad 1: VBATT_GATED -> /io_expander/GPB0
- U6 pad 2: GND -> /io_expander/GPB1
- U6 pad 3: 5V_GATED -> /io_expander/GPB2
- U6 pad 4: unconnected-(U6-Pad4) -> /io_expander/GPB3
- U6 pad 5: /power_cutoff/5V_EN -> /io_expander/GPB4
- U6 pad 6: unconnected-(U6-Pad6) -> /io_expander/GPB5
- U7 pad 1: Net-(R12-Pad1) -> unconnected-(U7-Pad1)
- U7 pad 10: /SCL -> unconnected-(U7-Pad10)
- U7 pad 2: Net-(R11-Pad2) -> unconnected-(U7-Pad2)
- U7 pad 4: /ADS0 -> /ESP32_Module/USB_DP
- U7 pad 5: /ADC/ADS_IN1 -> /ESP32_Module/USB_DN
- U7 pad 6: /ADS2 -> 3V3_GATED
- U7 pad 7: /ADC/ADS_IN3 -> 3V3_GATED
- U7 pad 8: 3V3_ESP32 -> Net-(C13-Pad1)
- U7 pad 9: /SDA -> Net-(R29-Pad2)
Routing:
- net +3V3: track 183.1 -> 0.00 mm, vias 3 -> 0
- net VBATT_GATED: track 141.2 -> 0.00 mm, vias 17 -> 0
- net 3V3_ESP32: track 107.9 -> 0.00 mm, vias 2 -> 0
- net /VBATT_trigger: track 81.2 -> 0.00 mm
- net /ESPIO16: track 77.4 -> 0.00 mm
- net 5V_GATED: track 74.0 -> 0.00 mm
- net /M1enc1: track 73.7 -> 0.00 mm
- net /M1enc2: track 67.7 -> 0.00 mm
- net +BATT: track 66.5 -> 0.00 mm
- net /ESPIO13: track 58.1 -> 0.00 mm, vias 1 -> 0
- net /ESPIO17: track 56.9 -> 0.00 mm
- net /ADC/ADS_IN1: track 56.7 -> 0.00 mm, vias 2 -> 0
- net /M1PWM2: track 56.6 -> 0.00 mm
- net /M1PWM1: track 51.0 -> 0.00 mm
- net /M2enc1: track 49.3 -> 0.00 mm
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- removed copper zone on B.Cu, net GND
- removed copper zone on F.Cu, net GND
Other:
- board size 97 x 57 mm -> 100 x 80 mm
- board text removed: "12V"
- board text removed: "12V 5V Gated"
- board text removed: "12V IN"
- board text removed: "3V3"
- board text removed: "5V"
- board text removed: "ADS1"
- board text removed: "ADS2"
- board text removed: "Boot"
- board text removed: "CLK"
- board text removed: "CS"
- board text removed: "E1"
- board text removed: "E18 RST"
- board text removed: "E18DC"
- board text removed: "E18DD"
- board text removed: "E18P10"
- board text removed: "E18P12"
- board text removed: "E18P14"
- board text removed: "E18P16"
- board text removed: "E18P17"
- board text removed: "E18RX"
- board text removed: "E18TX"
- board text removed: "E2"
- board text removed: "ESP EN"
- board text removed: "ESP32 devkitC V4"
- board text removed: "EXT1"
- board text removed: "G13"
- board text removed: "G15"
- board text removed: "G16"
- board text removed: "G17"
- board text removed: "G39"
- board text removed: "G4"
- board text removed: "GND"
- board text removed: "GPIO"
- board text removed: "I2C"
- board text removed: "M+"
- board text removed: "M-"
- board text removed: "MISO"
- board text removed: "MOSI"
- board text removed: "Motor1"
- board text removed: "Motor2"
- board text removed: "RXD0"
- board text removed: "SCL"
- board text removed: "SDA"
- board text removed: "SPI"
- board text removed: "TXD0"
- board text removed: "VBATT maintain"
- board text removed: "VBATT trig"
