File: Projects/Pippino_board_v2/pippino_board/pippino_board.kicad_sch (KiCad schematic)
At the start: 24 parts, among them J1 Conn_02x01, J10 Conn_01x06, J11 Conn_01x02, J2 Conn_02x02_Counter_Clockwise, J3 Conn_02x07_Odd_Even, J4 Conn_01x04, J5 Conn_01x06, J6 Conn_01x04, J7 Conn_01x04, J8 Conn_01x04, J9 Conn_01x06, SW1 SW_Push, U1 ESP32-DevKitC, U2 Mini360, U3 E18-MS1-PCB

Commit message: added pippino board v2
Parts:
- removed C7: 47uF, Capacitor_SMD:CP_Elec_6.3x5.4, symbol Device:C_Polarized
- removed C8: 100nF, Capacitor_SMD:C_0805_2012Metric, symbol Device:C
- removed J11: Conn_01x02, Connector_PinHeader_2.54mm:PinHeader_1x02_P2.54mm_Horizontal, symbol Connector_Generic:Conn_01x02
- removed J3: Conn_02x07_Odd_Even, Connector_PinHeader_2.54mm:PinHeader_2x07_P2.54mm_Vertical, symbol Connector_Generic:Conn_02x07_Odd_Even
- removed J4, J8: Conn_01x04, Connector_PinHeader_2.54mm:PinHeader_1x04_P2.54mm_Vertical, symbol Connector_Generic:Conn_01x04
- removed U1: ESP32-DevKitC, ESP32-DevKitC:DIP2600W100P254L5400H500Q38N, symbol ESP32-DevKitC:ESP32-DevKitC
- removed U2: Mini360, Mini-360:Mini360, symbol mini360:Mini360
- added C1: 10uF, Capacitor_SMD:C_0805_2012Metric, symbol Device:C
- added D1, D2, D3, D4: LED, LED_SMD:LED_1206_3216Metric, symbol Device:LED
- added J10, J11: Conn_02x03, Connector_PinHeader_2.54mm:PinHeader_2x03_P2.54mm_Vertical_SMD, symbol Connector_Generic:Conn_02x03_Odd_Even
- added J2: Conn_02x09_Odd_Even, Connector_PinHeader_2.54mm:PinHeader_2x09_P2.54mm_Vertical_SMD, symbol Connector_Generic:Conn_02x14_Odd_Even
- added J3: Conn_01x04, Connector_PinHeader_2.54mm:PinHeader_1x04_P2.54mm_Vertical_SMD_Pin1Left, symbol Connector_Generic:Conn_01x04
- added R1, R2, R3, R4: 330, Resistor_SMD:R_1206_3216Metric, symbol Device:R
- C2: renamed from C9; value 47uF -> 470uF; footprint Capacitor_SMD:CP_Elec_6.3x5.4 -> Capacitor_SMD:CP_Elec_10x10.5
- J4: renamed from J5; footprint Connector_PinHeader_2.54mm:PinHeader_1x06_P2.54mm_Vertical -> Connector_PinHeader_2.54mm:PinHeader_1x06_P2.54mm_Vertical_SMD_Pin1Left
- J6, J7: footprint Connector_PinHeader_2.54mm:PinHeader_1x04_P2.54mm_Vertical -> Connector_PinHeader_2.54mm:PinHeader_1x04_P2.54mm_Vertical_SMD_Pin1Left
- renumbered D1 to D5, J2 to J5, J9 to J8, J10 to J9, R2 to R5, R3 to R6, R4 to R7, U3 to U1
Connections:
- net +3V3: now also C1.1, J2.1 (Pin_1), J2.28 (Pin_28), J3.1 (Pin_1)
- net ADS0: now also J2.6 (Pin_6)
- net ADS2: now also J2.8 (Pin_8)
- net E18DC: now also J2.16 (Pin_16)
- net E18DD: now also J2.14 (Pin_14)
- net E18P10: now also JP2.3 (B)
- net E18P14: now also J2.5 (Pin_5)
- net E18P15: now also J2.7 (Pin_7)
- net E18P16: now also J2.9 (Pin_9)
- net E18RST: now also J2.12 (Pin_12)
- net E18RX: now also J2.11 (Pin_11)
- net E18TX: now also J2.13 (Pin_13)
- net ESPEN: now also J2.4 (Pin_4)
- net ESPIO13: now also J6.2 (Pin_2)
- net EXT1: now also J2.3 (Pin_3)
- net GND: now also C1.2, J10.1 (Pin_1), J11.1 (Pin_1), J2.2 (Pin_2), J2.25 (Pin_25), J2.27 (Pin_27), J3.4 (Pin_4), R1.2, R2.2, R3.2, R4.2
- net M1PWM1: now also J10.4 (Pin_4)
- net M1enc1: now also J10.2 (Pin_2)
- net M2PWM1: now also J11.4 (Pin_4)
- net M2enc1: now also J11.2 (Pin_2)
- net RXD0: now also J2.23 (Pin_23)
- net TXD0: now also J2.21 (Pin_21)
- net VBATT_GATED: now also J10.3 (Pin_3), J11.3 (Pin_3)
- net RUN_LED: now reaches U1.12 (P1.3)
- net RUN_LED: now also J2.22 (Pin_22)
- net 3V3_ESP32 renamed 3V3_GATED
- net 5V_GATED renamed 5V0_GATED
- net E18P12 renamed NWK_LED
- net NWK_LED: now also J2.20 (Pin_20)
- net E18P17 renamed Batt_Low_Flag
- net Batt_Low_Flag: now also J2.18 (Pin_18); no longer JP2.3 (B)
- net ESPIO16 renamed ESPIO35
- net ESPIO35: now also J2.19 (Pin_19); no longer J6.2 (Pin_2)
- net ESPIO17 renamed ESPIO14
- net M1enc2 renamed M1enc2_dir
- net M1enc2_dir: now also J10.5 (Pin_5)
- net M2enc2 renamed M2enc2_dir
- net M2enc2_dir: now also J11.5 (Pin_5)
- new net: D2.1 (K), R2.1
- new net: D3.1 (K), R3.1
- new net: D1.1 (K), R1.1
- new net: D4.1 (K), R4.1
- new net ADS3: J2.10 (Pin_10)
- new net ESPIO1: J2.15 (Pin_15)
- new net ESPIO11: J3.2 (Pin_2)
- new net ESPIO12: J3.3 (Pin_3)
- new net ESPIO19: D3.2 (A)
- new net ESPIO2: J2.17 (Pin_17)
- new net ESPIO20: D4.2 (A)
- new net LED1: D1.2 (A), J2.24 (Pin_24)
- new net LED2: D2.2 (A), J2.26 (Pin_26)
- new net M1PWM2_brake: J10.6 (Pin_6)
- new net M2PWM2_brake: J11.6 (Pin_6)
- no-connect marks 19 -> 10
Other:
- sheet power_cutoff renamed PSU_Gated
- added sheet ESP32_Module (esp32_module.kicad_sch)
- added sheet PSU_3v3_BATT (psu_3v3_batt.kicad_sch)
- added sheet io_expander (io_expander.kicad_sch)
- sheet PSU_Gated: file power_cutoff.kicad_sch -> psu_gated.kicad_sch
- sheet PSU_Gated ports: added 3V3_GATED; removed none
- moved on the sheet: C2, D5, J1, J4, J7, J8, J9, R5
