File: Projects/Hydroponics_board_v1/Hydroponics_board_v1.kicad_pcb (KiCad board)
At the start: 2 copper layers, 100 x 90 mm, 73 parts, among them J1 Display, J10 EC_ANA, J11 WLEV_ANA, J12 ANA3, J13 IO, J14 Relays, J15 Buttons, J16 12V Power, J17 DCM0, J18 DCM1, J19 DCM2, J2 Flow Counter, J20 DCM3, J21 12V Power, J3 Onewire T, J4 GPIO, J5 I2C, J6 Step1, J7 Step2, J8 Step3, J9 PH_ANA, U1 ESP32-DevKitC, U10 DRV8833_M23, U11 ESP01, U2 Step Ctrl 1, U3 Step Ctrl 2, U4 Step Ctrl 3, U5 ADC, U6 MCP23017, U7 3.3V DC-DC, U8 5V DC-DC, U9 DRV8833_M01

Commit message: work on pippino board v2
Changed lines of the file:
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@@
     (property "Sheetfile" "stepper_pump_ctrl.kicad_sch")
     (property "Sheetname" "stepper_pump_control")
-    (zone_connect 2)
     (attr through_hole)
     (fp_text reference "U3" (at 0.253 0.762 180) (layer "F.SilkS")
@@
     (property "Sheetfile" "stepper_pump_ctrl.kicad_sch")
     (property "Sheetname" "stepper_pump_control")
-    (zone_connect 2)
     (attr through_hole)
     (fp_text reference "U2" (at 0.253 1.387 180) (layer "F.SilkS")
@@
     (property "Sheetfile" "pwm_pump_ctrl.kicad_sch")
     (property "Sheetname" "PWM_motor_control")
+    (zone_connect 2)
     (attr smd)
     (fp_text reference "U9" (at 0 -3.45) (layer "F.SilkS")
@@
     (property "Sheetfile" "stepper_pump_ctrl.kicad_sch")
     (property "Sheetname" "stepper_pump_control")
-    (zone_connect 2)
     (attr through_hole)
     (fp_text reference "U4" (at 0.38 0.508 180) (layer "F.SilkS")
@@
     (property "Sheetfile" "pwm_pump_ctrl.kicad_sch")
     (property "Sheetname" "PWM_motor_control")
+    (zone_connect 2)
     (attr smd)
     (fp_text reference "U10" (at 0 -3.45) (layer "F.SilkS")
@@
     (property "Sheetfile" "Hydroponics_board_v1.kicad_sch")
     (property "Sheetname" "")
-    (zone_connect 2)
+    (zone_connect 1)
     (attr through_hole)
     (fp_text reference "U1" (at 0 -2.54) (layer "F.SilkS")
@@
     (effects (font (size 1 1) (thickness 0.15)))
   )
-  (gr_text "3v3" (at 157.48 60.96 90) (layer "F.SilkS")
+  (gr_text "3v3" (at 157.48 66.548 90) (layer "F.SilkS")
     (effects (font (size 1 1) (thickness 0.15)))
   )
@@
     (effects (font (size 1 1) (thickness 0.15)))
   )
-  (gr_text "WL" (at 157.48 64.008 90) (layer "F.SilkS")
+  (gr_text "WL" (at 157.48 63.5 90) (layer "F.SilkS")
     (effects (font (size 1 1) (thickness 0.15)))
   )
-  (gr_text "G" (at 157.48 66.548 90) (layer "F.SilkS")
+  (gr_text "G" (at 157.48 60.96 90) (layer "F.SilkS")
     (effects (font (size 1 1) (thickness 0.15)))
   )
@@
   (segment (start 77.470001 75.689999) (end 74.424001 75.689999) (width 4) (layer "F.Cu") (net 1))
   (segment (start 69.5 72) (end 69.5 73.5) (width 4) (layer "F.Cu") (net 1))
-  (segment (start 76.948489 51.490511) (end 76.948489 48.26) (width 4) (layer "F.Cu") (net 1))
+  (segment (start 76.2 51.490511) (end 76.2 48.26) (width 4) (layer "F.Cu") (net 1))
   (segment (start 100.1776 44.0436) (end 100.1776 42.3224) (width 2) (layer "F.Cu") (net 1))
   (segment (start 78.486 86.868) (end 81.026 89.408) (width 4) (layer "F.Cu") (net 1))
@@
   (segment (start 120.690489 42.190489) (end 122.25 43.75) (width 3.5) (layer "F.Cu") (net 1))
   (segment (start 76.708 85.09) (end 78.486 86.868) (width 4) (layer "F.Cu") (net 1))
-  (segment (start 76.948489 48.26) (end 77 45.5) (width 4) (layer "F.Cu") (net 1))
+  (segment (start 76.2 48.26) (end 76.251511 45.5) (width 4) (layer "F.Cu") (net 1))
   (segment (start 76.948489 44.551511) (end 77.5 44) (width 4) (layer "F.Cu") (net 1))
   (segment (start 76.073 84.455) (end 72.898 81.28) (width 4) (layer "F.Cu") (net 1))
@@
   (segment (start 100.309511 43.911689) (end 100.309511 42.190489) (width 2) (layer "B.Cu") (net 1))
   (segment (start 72.449512 75.689999) (end 69.399511 78.74) (width 4) (layer "B.Cu") (net 1))
+  (segment (start 74.9695 53.4695) (end 76.2 52.239) (width 4) (layer "B.Cu") (net 1))
   (segment (start 71.636 54.864) (end 73.575 54.864) (width 4) (layer "B.Cu") (net 1))
-  (segment (start 76.948489 51.490511) (end 76.948489 48.26) (width 4) (layer "B.Cu") (net 1))
   (segment (start 73.575 54.864) (end 73.7195 54.7195) (width 4) (layer "B.Cu") (net 1))
   (segment (start 100.2284 43.9928) (end 100.309511 43.911689) (width 2) (layer "B.Cu") (net 1))
@@
   (segment (start 79.309511 42.190489) (end 100.190489 42.190489) (width 3.5) (layer "B.Cu") (net 1))
   (segment (start 89.845 103.5) (end 93.02 100.325) (width 8) (layer "B.Cu") (net 1))
-  (segment (start 74.9695 53.4695) (end 76.948489 51.490511) (width 4) (layer "B.Cu") (net 1))
   (segment (start 70.612 78.74) (end 73.279 81.407) (width 4) (layer "B.Cu") (net 1))
   (segment (start 100.190489 44.030711) (end 100.2284 43.9928) (width 4) (layer "B.Cu") (net 1))
   (segment (start 68.275 54.864) (end 71.636 54.864) (width 4) (layer "B.Cu") (net 1))
   (segment (start 100.190489 52.190489) (end 101 53) (width 4) (layer "B.Cu") (net 1))
-  (segment (start 76.948489 48.26) (end 76.948489 44.551511) (width 4) (layer "B.Cu") (net 1))
+  (segment (start 76.2 45.3) (end 76.948489 44.551511) (width 4) (layer "B.Cu") (net 1))
   (segment (start 73.7195 54.7195) (end 74.9695 53.4695) (width 4) (layer "B.Cu") (net 1))
   (segment (start 77.470001 88.389999) (end 78.488002 89.408) (width 4) (layer "B.Cu") (net 1))
@@
   (segment (start 73.575 64.115) (end 73.575 54.864) (width 4) (layer "B.Cu") (net 1))
   (segment (start 93.472 97.79) (end 93.472 98.298) (width 6) (layer "B.Cu") (net 1))
+  (segment (start 76.2 52.239) (end 76.2 45.3) (width 4) (layer "B.Cu") (net 1))
   (segment (start 78.4175 114.005) (end 80.005 114.005) (width 0.25) (layer "F.Cu") (net 2))
   (segment (start 83.955 97.225) (end 84.93 98.2) (width 0.25) (layer "F.Cu") (net 2))
