File: Projects/Hydroponics_board_v1/Hydroponics_board_v1.kicad_sch (KiCad schematic)
At the start: 8 parts, among them J1 Display, J2 Flow Counter, J3 Onewire T, J4 GPIO, J5 I2C, U1 ESP32-DevKitC, U11 ESP01

Commit message: work on pippino board v2
Connections:
- net m1_in1: now also U1.11 (IO27); no longer U1.13 (IO12)
- net m1_in2: now also U1.13 (IO12); no longer U1.11 (IO27)
- net m3_in1: now also U1.8 (IO33); no longer U1.7 (IO32)
- net m3_in2: now also U1.7 (IO32); no longer U1.8 (IO33)
Changed lines of the file:
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@@
     (effects (font (size 1.27 1.27)) (justify right bottom))
   )
-  (label "m1_in2" (at 91.44 63.5 0)
+  (label "m1_in2" (at 91.44 68.58 0)
     (effects (font (size 1.27 1.27)) (justify left bottom))
   )
@@
     (effects (font (size 1.27 1.27)) (justify left bottom))
   )
-  (label "m1_in1" (at 91.44 68.58 0)
+  (label "m1_in1" (at 91.44 63.5 0)
     (effects (font (size 1.27 1.27)) (justify left bottom))
   )
@@
     (effects (font (size 1.27 1.27)) (justify left bottom))
   )
-  (label "m3_in2" (at 91.44 55.88 0)
+  (label "m3_in2" (at 91.44 53.34 0)
     (effects (font (size 1.27 1.27)) (justify left bottom))
   )
@@
     (effects (font (size 1.27 1.27)) (justify left bottom))
   )
-  (label "m3_in1" (at 91.44 53.34 0)
+  (label "m3_in1" (at 91.44 55.88 0)
     (effects (font (size 1.27 1.27)) (justify left bottom))
   )
@@
       (reference "#PWR037") (unit 1) (value "GND") (footprint "")
     )
-    (path "/a44440a4-68f0-4517-92c3-20a982c3dffa/54f2aadc-6c67-45f7-a995-192b30cba7d0"
-      (reference "#PWR038") (unit 1) (value "+3V3") (footprint "")
-    )
     (path "/a44440a4-68f0-4517-92c3-20a982c3dffa/3d6cdd62-5634-4e30-acf8-1b9c1dbf6653"
