File: Projects/Hydroponics_board_v1/analog_sensors.kicad_sch (KiCad schematic)
At the start: 13 parts, among them J10 EC_ANA, J11 WLEV_ANA, J12 ANA3, J9 PH_ANA, U5 ADC

Commit message: work on pippino board v2
Connections:
- net +3V3: no longer C5.1, R2.1, R4.1, R5.1, U5.8 (VDD)
- net at C4.1, FB1.2: now also C5.1, R2.1, R4.1, R5.1, U5.8 (VDD)
Other:
- moved on the sheet: C4, FB1, FB2
Changed lines of the file:
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@@
   (junction (at 140.97 41.91) (diameter 0) (color 0 0 0 0)
   )
+  (junction (at 46.99 41.91) (diameter 0) (color 0 0 0 0)
+  )
+  (junction (at 102.87 41.91) (diameter 0) (color 0 0 0 0)
+  )
   (junction (at 119.38 41.91) (diameter 0) (color 0 0 0 0)
   )
   (junction (at 130.81 64.77) (diameter 0) (color 0 0 0 0)
   )
-  (junction (at 102.87 41.91) (diameter 0) (color 0 0 0 0)
-  )
   (junction (at 140.97 67.31) (diameter 0) (color 0 0 0 0)
   )
@@
     (stroke (width 0) (type default) (color 0 0 0 0))
   )
-  (wire (pts (xy 43.18 85.09) (xy 43.18 76.2))
+  (wire (pts (xy 46.99 68.58) (xy 46.99 59.69))
     (stroke (width 0) (type default) (color 0 0 0 0))
   )
@@
     (stroke (width 0) (type default) (color 0 0 0 0))
   )
-  (wire (pts (xy 43.18 59.69) (xy 43.18 55.88))
-    (stroke (width 0) (type default) (color 0 0 0 0))
-  )
-  (wire (pts (xy 43.18 67.31) (xy 43.18 71.12))
+  (wire (pts (xy 46.99 50.8) (xy 46.99 54.61))
+    (stroke (width 0) (type default) (color 0 0 0 0))
+  )
+  (wire (pts (xy 46.99 39.37) (xy 46.99 41.91))
     (stroke (width 0) (type default) (color 0 0 0 0))
   )
@@
     (stroke (width 0) (type default) (color 0 0 0 0))
   )
-  (wire (pts (xy 102.87 39.37) (xy 102.87 41.91))
+  (wire (pts (xy 46.99 41.91) (xy 102.87 41.91))
     (stroke (width 0) (type default) (color 0 0 0 0))
   )
@@
     (stroke (width 0) (type default) (color 0 0 0 0))
   )
+  (wire (pts (xy 46.99 41.91) (xy 46.99 43.18))
+    (stroke (width 0) (type default) (color 0 0 0 0))
+  )
   (wire (pts (xy 132.08 116.84) (xy 138.43 116.84))
     (stroke (width 0) (type default) (color 0 0 0 0))
@@
     (stroke (width 0) (type default) (color 0 0 0 0))
   )
-  (wire (pts (xy 43.18 41.91) (xy 43.18 50.8))
+  (wire (pts (xy 46.99 25.4) (xy 46.99 34.29))
     (stroke (width 0) (type default) (color 0 0 0 0))
   )
@@
     (pin "3")
   )
-  (symbol (lib_id "power:+3V3") (at 43.18 41.91 0) (unit 1)
-    (in_bom yes) (on_board yes) (fields_autoplaced)
-    (property "Reference" "#PWR034" (id 0) (at 43.18 45.72 0)
-      (effects (font (size 1.27 1.27)) hide)
-    )
-    (property "Value" "+3V3" (id 1) (at 43.18 36.83 0))
-    (property "Footprint" "" (id 2) (at 43.18 41.91 0)
-      (effects (font (size 1.27 1.27)) hide)
-    )
-    (property "Datasheet" "" (id 3) (at 43.18 41.91 0)
+  (symbol (lib_id "power:+3V3") (at 46.99 25.4 0) (unit 1)
+    (in_bom yes) (on_board yes) (fields_autoplaced)
+    (property "Reference" "#PWR034" (id 0) (at 46.99 29.21 0)
+      (effects (font (size 1.27 1.27)) hide)
+    )
+    (property "Value" "+3V3" (id 1) (at 46.99 20.32 0))
+    (property "Footprint" "" (id 2) (at 46.99 25.4 0)
+      (effects (font (size 1.27 1.27)) hide)
+    )
+    (property "Datasheet" "" (id 3) (at 46.99 25.4 0)
       (effects (font (size 1.27 1.27)) hide)
     )
@@
     (pin "1")
   )
-  (symbol (lib_id "Device:FerriteBead_Small") (at 43.18 53.34 0) (unit 1)
-    (in_bom yes) (on_board yes) (fields_autoplaced)
-    (property "Reference" "FB1" (id 0) (at 45.72 52.0318 0)
-      (effects (font (size 1.27 1.27)) (justify left))
-    )
-    (property "Value" "FerriteBead_Small" (id 1) (at 45.72 54.5718 0)
-      (effects (font (size 1.27 1.27)) (justify left))
-    )
-    (property "Footprint" "Resistor_SMD:R_1206_3216Metric" (id 2) (at 41.402 53.34 90)
-      (effects (font (size 1.27 1.27)) hide)
-    )
-    (property "Datasheet" "~" (id 3) (at 43.18 53.34 0)
-      (effects (font (size 1.27 1.27)) hide)
-    )
-    (pin "1")
-    (pin "2")
-  )
-  (symbol (lib_id "power:+3V3") (at 102.87 39.37 0) (unit 1)
-    (in_bom yes) (on_board yes) (fields_autoplaced)
-    (property "Reference" "#PWR038" (id 0) (at 102.87 43.18 0)
-      (effects (font (size 1.27 1.27)) hide)
-    )
-    (property "Value" "+3V3" (id 1) (at 102.87 34.29 0))
-    (property "Footprint" "" (id 2) (at 102.87 39.37 0)
-      (effects (font (size 1.27 1.27)) hide)
-    )
-    (property "Datasheet" "" (id 3) (at 102.87 39.37 0)
-      (effects (font (size 1.27 1.27)) hide)
-    )
-    (pin "1")
+  (symbol (lib_id "Device:FerriteBead_Small") (at 46.99 36.83 0) (unit 1)
+    (in_bom yes) (on_board yes) (fields_autoplaced)
+    (property "Reference" "FB1" (id 0) (at 49.53 35.5218 0)
+      (effects (font (size 1.27 1.27)) (justify left))
+    )
+    (property "Value" "FerriteBead_Small" (id 1) (at 49.53 38.0618 0)
+      (effects (font (size 1.27 1.27)) (justify left))
+    )
+    (property "Footprint" "Resistor_SMD:R_1206_3216Metric" (id 2) (at 45.212 36.83 90)
+      (effects (font (size 1.27 1.27)) hide)
+    )
+    (property "Datasheet" "~" (id 3) (at 46.99 36.83 0)
+      (effects (font (size 1.27 1.27)) hide)
+    )
+    (pin "1")
+    (pin "2")
   )
   (symbol (lib_id "Device:R") (at 140.97 52.07 0) (unit 1)
@@
     (pin "2")
   )
-  (symbol (lib_id "power:GND") (at 43.18 85.09 0) (unit 1)
-    (in_bom yes) (on_board yes) (fields_autoplaced)
-    (property "Reference" "#PWR035" (id 0) (at 43.18 91.44 0)
-      (effects (font (size 1.27 1.27)) hide)
-    )
-    (property "Value" "GND" (id 1) (at 43.18 90.17 0))
-    (property "Footprint" "" (id 2) (at 43.18 85.09 0)
-      (effects (font (size 1.27 1.27)) hide)
-    )
-    (property "Datasheet" "" (id 3) (at 43.18 85.09 0)
+  (symbol (lib_id "power:GND") (at 46.99 68.58 0) (unit 1)
+    (in_bom yes) (on_board yes) (fields_autoplaced)
+    (property "Reference" "#PWR035" (id 0) (at 46.99 74.93 0)
+      (effects (font (size 1.27 1.27)) hide)
+    )
+    (property "Value" "GND" (id 1) (at 46.99 73.66 0))
+    (property "Footprint" "" (id 2) (at 46.99 68.58 0)
+      (effects (font (size 1.27 1.27)) hide)
+    )
+    (property "Datasheet" "" (id 3) (at 46.99 68.58 0)
       (effects (font (size 1.27 1.27)) hide)
     )
@@
     (pin "1")
   )
-  (symbol (lib_id "Device:C") (at 43.18 63.5 0) (unit 1)
-    (in_bom yes) (on_board yes) (fields_autoplaced)
-    (property "Reference" "C4" (id 0) (at 46.99 62.2299 0)
-      (effects (font (size 1.27 1.27)) (justify left))
-    )
-    (property "Value" "1uF" (id 1) (at 46.99 64.7699 0)
-      (effects (font (size 1.27 1.27)) (justify left))
-    )
-    (property "Footprint" "Capacitor_SMD:C_0805_2012Metric" (id 2) (at 44.1452 67.31 0)
-      (effects (font (size 1.27 1.27)) hide)
-    )
-    (property "Datasheet" "~" (id 3) (at 43.18 63.5 0)
+  (symbol (lib_id "Device:C") (at 46.99 46.99 0) (unit 1)
+    (in_bom yes) (on_board yes) (fields_autoplaced)
+    (property "Reference" "C4" (id 0) (at 50.8 45.7199 0)
+      (effects (font (size 1.27 1.27)) (justify left))
+    )
+    (property "Value" "1uF" (id 1) (at 50.8 48.2599 0)
+      (effects (font (size 1.27 1.27)) (justify left))
+    )
+    (property "Footprint" "Capacitor_SMD:C_0805_2012Metric" (id 2) (at 47.9552 50.8 0)
+      (effects (font (size 1.27 1.27)) hide)
+    )
+    (property "Datasheet" "~" (id 3) (at 46.99 46.99 0)
       (effects (font (size 1.27 1.27)) hide)
     )
@@
     (pin "3")
   )
-  (symbol (lib_id "Device:FerriteBead_Small") (at 43.18 73.66 0) (unit 1)
-    (in_bom yes) (on_board yes) (fields_autoplaced)
-    (property "Reference" "FB2" (id 0) (at 45.72 72.3518 0)
-      (effects (font (size 1.27 1.27)) (justify left))
-    )
-    (property "Value" "FerriteBead_Small" (id 1) (at 45.72 74.8918 0)
-      (effects (font (size 1.27 1.27)) (justify left))
-    )
-    (property "Footprint" "Resistor_SMD:R_1206_3216Metric" (id 2) (at 41.402 73.66 90)
-      (effects (font (size 1.27 1.27)) hide)
-    )
-    (property "Datasheet" "~" (id 3) (at 43.18 73.66 0)
-      (effects (font (size 1.27 1.27)) hide)
-    )
+  (symbol (lib_id "Device:FerriteBead_Small") (at 46.99 57.15 0) (unit 1)
+    (in_bom yes) (on_board yes) (fields_autoplaced)
+    (property "Reference" "FB2" (id 0) (at 49.53 55.8418 0)
+      (effects (font (size 1.27 1.27)) (justify left))
+    )
+    (property "Value" "FerriteBead_Small" (id 1) (at 49.53 58.3818 0)
+      (effects (font (size 1.27 1.27)) (justify left))
+    )
+    (property "Footprint" "Resistor_SMD:R_1206_3216Metric" (id 2) (at 45.212 57.15 90)
+      (effects (font (size 1.27 1.27)) hide)
+    )
+    (property "Datasheet" "~" (id 3) (at 46.99 57.15 0)
+      (effects (font (size 1.27 1.27)) hide)
+    )
