File: Projects/Hydroponics_board_v1/pwm_pump_ctrl.kicad_sch (KiCad schematic)
At the start: 14 parts, among them J17 DCM0, J18 DCM1, J19 DCM2, J20 DCM3, U10 DRV8833_M23, U9 DRV8833_M01

Commit message: work on pippino board v2
Connections:
- net m1_in1: now also JP8.1 (A); no longer JP7.1 (A)
- net m1_in2: now also JP7.1 (A); no longer JP8.1 (A)
- net m3_in1: now also U10.10 (BIN2); no longer U10.9 (BIN1)
- net m3_in2: now also U10.9 (BIN1); no longer U10.10 (BIN2)
Changed lines of the file:
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@@
     (effects (font (size 1.27 1.27)) (justify left bottom))
   )
-  (hierarchical_label "m1_in2" (shape input) (at 67.31 133.35 180)
+  (hierarchical_label "m1_in1" (shape input) (at 67.31 133.35 180)
     (effects (font (size 1.27 1.27)) (justify right))
   )
@@
     (effects (font (size 1.27 1.27)) (justify right))
   )
-  (hierarchical_label "m1_in1" (shape input) (at 38.1 133.35 180)
+  (hierarchical_label "m1_in2" (shape input) (at 38.1 133.35 180)
     (effects (font (size 1.27 1.27)) (justify right))
   )
@@
     (effects (font (size 1.27 1.27)) (justify right))
   )
-  (hierarchical_label "m3_in1" (shape input) (at 195.58 115.57 180)
+  (hierarchical_label "m3_in1" (shape input) (at 195.58 118.11 180)
     (effects (font (size 1.27 1.27)) (justify right))
   )
@@
     (effects (font (size 1.27 1.27)) (justify right))
   )
-  (hierarchical_label "m3_in2" (shape input) (at 195.58 118.11 180)
+  (hierarchical_label "m3_in2" (shape input) (at 195.58 115.57 180)
     (effects (font (size 1.27 1.27)) (justify right))
   )
