File: Projects/Pippino_board_brushless_v2/pippino_board/tps_62110_module_batt.kicad_sch (KiCad schematic)
At the start: 11 parts, among them U8 TPS62110

Commit message: work on pippino board v2
Parts:
- R34: value 720K -> 680K
Other:
- note added: "Battery low triggers at: 1.256V/100K*(680K+100K) = 9.8 V"
