File: Projects/Pippino_board_brushless_v2/pippino_board/pippino_board.kicad_pcb (KiCad board)
At the start: 2 copper layers, 100 x 80 mm, 103 parts, among them J1 Conn_02x06_Odd_Even, J10 USB_B_Micro, J2 Conn_02x01, J3 Conn_02x06_Odd_Even, J4 Conn_02x02_Counter_Clockwise, J5 Conn_02x09_Odd_Even, J6 Conn_02x03, J7 Conn_02x03, J8 Conn_02x02_Odd_Even, J9 IO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

Commit message: work on pippino board v2
Other:
- board text added: "locked"
- board text removed: "BRK"
- board text removed: "DIR"
- board text removed: "E18P10"
- board text removed: "E18P16"
- board text removed: "ENC"
- board text removed: "ESP13"
- board text removed: "M1"
- board text removed: "M2"
- board text removed: "MAINTAIN"
- board text removed: "PWM"
- board text removed: "TRIGGER"

Commit message: work on pcb
Parts:
- R34: value 720K -> 680K
- moved R21 2.06 mm to (150.2, 135.2)
- moved R35 2.01 mm to (152.8, 135.2)
- moved J10 0.33 mm to (112.3, 154.2)
- turned Q1 to 0 degrees
Routing:
- net /ESP32_Module/GPIO0: track 72.8 -> 86.6 mm, vias 2 -> 6
- net VBATT_GATED: track 102.4 -> 97.5 mm, vias 4 -> 0
- net +BATT: track 38.2 -> 34.5 mm, vias 2 -> 0
- net GND: track 8.46 -> 11.1 mm, vias 167 -> 255
- net /PSU_3v3_BATT/TPS62110_MODULE_BATT/FB_1v15: track 20.6 -> 18.0 mm
- net /VBATT_trigger: track 34.6 -> 32.4 mm
- net /ADC/ADS_IN2: track 47.8 -> 45.7 mm
- net /3v3_PWR_Good: track 57.5 -> 55.7 mm
- net /Batt_Low_Flag: track 145.2 -> 143.7 mm, vias 3 -> 5
- net /SCL: track 71.2 -> 69.8 mm
- net Net-(Q1-C): track 14.5 -> 13.2 mm
- net /SDA: track 72.2 -> 71.0 mm
- net /VBATT_maintain: track 31.6 -> 32.7 mm, vias 1 -> 2
- net /VBATT_trig_manual: track 47.6 -> 46.8 mm
