File: Projects/Pippino_board_brushless_v2/pippino_board/pippino_board.kicad_sch (KiCad schematic)
At the start: 31 parts, among them J1 Conn_02x06_Odd_Even, J2 Conn_02x01, J3 Conn_02x06_Odd_Even, J4 Conn_02x02_Counter_Clockwise, J5 Conn_02x09_Odd_Even, J6 Conn_02x03, J7 Conn_02x03, J8 Conn_02x02_Odd_Even, SW1 SW_Push, U1 E18-MS1-PCB

Commit message: work on pippino II board v2.1
Other:
- title: (none) -> Pippino II Schematic v2.0
Changed lines of the file:
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@@
 (kicad_sch (version 20230121) (generator eeschema)
   (paper "A4")
+  (title_block
+    (title "Pippino II Schematic v2.0")
+  )
   (junction (at 64.77 104.14) (diameter 0) (color 0 0 0 0)
   )
