File: Projects/Pippino_board_brushless_v2/pippino_board/psu_3v3.kicad_sch (KiCad schematic)
At the start: 2 parts

Commit message: work on pippino II board v2.1
Other:
- note added: "Wrong design, resistor divider should be at the VOUT"
Changed lines of the file:
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@@
     (stroke (width 0) (type default))
+  )
+  (text "Wrong design, resistor divider should be at the VOUT"
+    (at 123.19 67.31 0)
+    (effects (font (size 1.27 1.27)) (justify left bottom))
   )
   (hierarchical_label "3V3" (shape output) (at 175.26 83.82 0) (fields_autoplaced)
