File: Projects/Pippino_board_brushless_v2/pippino_board/psu_3v3_batt.kicad_sch (KiCad schematic)
At the start: 2 parts

Commit message: work on pippino II board v2.1
Other:
- note added: "Wrong design, resistor divider should be at the VOUT"
Changed lines of the file:
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@@
     (stroke (width 0) (type default))
+  )
+  (text "Wrong design, resistor divider should be at the VOUT"
+    (at 115.57 67.31 0)
+    (effects (font (size 1.27 1.27)) (justify left bottom))
   )
   (hierarchical_label "Power_Good_Flag" (shape output) (at 175.26 91.44 0) (fields_autoplaced)
