File: Projects/Pippino_board_brushless_v2.1/pippino_board/adc_block.kicad_sch (KiCad schematic)
At the start: 9 parts, among them U2 ADS1115IDGS

Commit message: moved to ubu 22, updated pippino v2.1
Parts:
- R16, R17, R18, R19: value 10k -> 10K
- U2: footprint Package_SO:TSSOP-10_3x3mm_P0.5mm -> Package_SO:VSSOP-10_3x3mm_P0.5mm
Other:
- moved on the sheet: C5, FB1, FB2
