File: Projects/Pippino_board_brushless_v2.1/pippino_board/esp32_module.kicad_sch (KiCad schematic)
At the start: 18 parts, among them J10 USB_B_Micro, Q3 L8050_SOT23, Q4 L8050_SOT23, SW2 SW_Push, U5 CP2102N-Axx-xQFN28, U6 ESP32-S3-WROOM-1

Commit message: work on pippino II board v2.1
Parts:
- R31: value 10K(NC) -> 10K
Connections:
- no-connect marks 31 -> 32

Commit message: moved to ubu 22, updated pippino v2.1
Connections:
- net GPIO45: now reaches U6.26 (GPIO45)
- no-connect marks 32 -> 30
Other:
- moved on the sheet: D10, D11, D12, J10
