File: Projects/Pippino_board_brushless_v2.1/pippino_board/pippino_board.kicad_pcb (KiCad board)
At the start: 2 copper layers, 181.3 x 80 mm, 104 parts, among them J1 Conn_02x06_Odd_Even, J10 USB_B_Micro, J11 Conn_02x01, J2 Conn_02x01, J3 Conn_02x06_Odd_Even, J4 Conn_02x02_Counter_Clockwise, J5 Conn_02x09_Odd_Even, J6 Conn_02x03, J7 Conn_02x03, J8 Conn_02x02_Odd_Even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

Commit message: work on pippino II board v2.1
Parts:
- R31: value 10K(NC) -> 10K
- U7: value CK1408 -> CK1418
- moved C19 13.3 mm to (138.1, 146.5), turned to 0 degrees
- moved C20 11.2 mm to (137.7, 144.2), turned to 0 degrees
- moved R7 6.17 mm to (197.5, 147.2)
- moved C10 5.30 mm to (166.0, 122.5), turned to 0 degrees
- moved R9 4.86 mm to (157.6, 135.5), turned to -90 degrees
- moved R35 2.96 mm to (151.5, 134.1)
- moved R21 2.92 mm to (149.0, 134.1)
- moved R8 2.21 mm to (162.8, 135.4), turned to 180 degrees
- moved R34 2.00 mm to (152.5, 141.5)
- moved R13 1.91 mm to (158.2, 139.2), turned to 180 degrees
- moved D7 1.12 mm to (197.5, 144.8), turned to 0 degrees
- moved R22 1.00 mm to (166.0, 125.0)
- moved R23 0.52 mm to (170.1, 120.0)
- moved C16 0.25 mm to (159.2, 142.2)
- moved C17 0.25 mm to (157.0, 142.2)
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Routing:
- net VBATT_GATED: track 96.9 -> 45.5 mm, vias 4 -> 0
- net +3V3: track 98.9 -> 91.4 mm
- net /VBATT_trigger: track 37.7 -> 32.0 mm, vias 1 -> 2
- net Net-(U3-PG): track 0.00 -> 4.34 mm
- net /Batt_Low_Flag: track 144.8 -> 140.8 mm
- net /ADC/ADS_IN2: track 48.4 -> 44.8 mm
- net /VBATT_trig_manual: track 46.8 -> 44.2 mm
- net 3V3_GATED: track 206.8 -> 209.2 mm
- net /3v3_PWR_Good: track 57.1 -> 54.7 mm
- net /ESP32_Module/DTR: track 31.6 -> 33.8 mm
- net +BATT: track 26.3 -> 28.3 mm
- net /ESP32_Module/GPIO0: track 82.0 -> 83.9 mm, vias 2 -> 6
- net 5V0_GATED: track 29.5 -> 31.3 mm, vias 13 -> 12
- net /PSU_Gated/PSU_3v3/TPS62110_MODULE/FB_1v15: track 11.6 -> 10.0 mm
- net /ADC/3V3_filtered: track 6.34 -> 7.50 mm
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Other:
- board size 181.3 x 80 mm -> 100 x 80 mm
- board text added: "PWR"
- board text removed: "POWER LED"

Commit message: moved to ubu 22, updated pippino v2.1
Parts:
- added D13: 1N5819, Diode_SMD:D_SOD-123, F.Cu at (145.0, 151.2)
- added J12: Conn_02x02_Odd_Even, Connector_PinHeader_2.54mm:PinHeader_2x02_P2.54mm_Vertical, F.Cu at (185.9, 114.0)
- added JP3: SolderJumper_2_Open, Jumper:SolderJumper-2_P1.3mm_Open_RoundedPad1.0x1.5mm, F.Cu at (191.6, 113.8)
- added R38: 360, Resistor_SMD:R_1206_3216Metric, F.Cu at (145.0, 153.8)
- added TP1: VBG, TestPoint:TestPoint_Pad_D1.5mm, F.Cu at (182.6, 142.4)
- added TP3: VB, TestPoint:TestPoint_Pad_D1.5mm, F.Cu at (171.2, 148.2)
- J1: footprint Connector_PinHeader_2.54mm:PinHeader_2x07_P2.54mm_Vertical -> Connector_PinHeader_2.54mm:PinHeader_2x08_P2.54mm_Vertical
- J5: value Conn_02x09_Odd_Even -> Conn_02x08_Odd_Even; footprint Connector_PinHeader_2.54mm:PinHeader_2x09_P2.54mm_Vertical -> Connector_PinHeader_2.54mm:PinHeader_2x08_P2.54mm_Vertical
- Q1: footprint Package_TO_SOT_SMD:SOT-23 -> Components:2N3904_SOT-23
- R10, R15: value 220K -> 200K
- R11, R14: value 220 -> 360
- R12: value 100K -> 200K
- R13: value 100k -> 200K
- R16, R17, R18, R19, R25, R26: value 10k -> 10K
- R7: value 330 -> 1K
- R8: value 18k -> 18K
- R9: value 5.1k -> 5.1K
- U2: footprint Package_SO:TSSOP-10_3x3mm_P0.5mm -> Package_SO:VSSOP-10_3x3mm_P0.5mm
- U7: value CK1418 -> CKCS_BK03; footprint Pcb_Modules:CK1408 -> Pcb_Modules:CKCS-BK03
- moved R7 30.4 mm to (194.2, 117.0), turned to 180 degrees
- moved D7 28.9 mm to (189.6, 117.0)
- moved R27 12.6 mm to (121.4, 148.2)
- moved SW1 6.16 mm to (140.5, 157.2), turned to 0 degrees
- moved MH3 6.00 mm to (196.0, 84.0)
- moved MH3 6.00 mm to (110.0, 84.0)
- moved MH3 6.00 mm to (196.0, 143.0)
- moved MH3 6.00 mm to (110.0, 143.0)
- moved R24 5.46 mm to (175.2, 129.0)
- moved R23 4.91 mm to (172.6, 124.2), turned to -90 degrees
- moved R32 4.16 mm to (132.2, 157.5), turned to 180 degrees
- moved J1 2.54 mm to (103.7, 91.8)
- moved D10 1.97 mm to (110.0, 147.2)
- moved Q4 1.91 mm to (139.8, 152.0), turned to 90 degrees
- moved U1 0.96 mm to (122.0, 92.1)
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Connections:
- D8 pad 1: /VBATT_trig_manual -> Net-(D13-K)
- D9 pad 1: /VBATT_trig_manual -> Net-(D13-K)
- J1 pad 10: /E18TX -> /E18P16
- J1 pad 11: /RUN_LED -> /E18RX
- J1 pad 12: /NWK_LED -> /E18TX
- J1 pad 13: /LED2 -> /RUN_LED
- J1 pad 14: /LED1 -> /NWK_LED
- J1 pad 3: /E18RST -> GND
- J1 pad 4: /E18DC -> +3V3
- J1 pad 5: /E18P14 -> /E18RST
- J1 pad 6: /E18DD -> /E18DC
- J1 pad 7: /E18P15 -> /E18P14
- J1 pad 8: /E18P16 -> /E18DD
- J1 pad 9: /E18RX -> /E18P15
- J11 pad 2: 5V0_GATED -> VBATT_GATED
- J5 pad 15: /ESPIO14 -> /ESPIO12
- J5 pad 16: /ESPIO48 -> /ESPIO14
- Q1 pad 1: /VBATT_trig_manual -> GND
- Q1 pad 2: GND -> Net-(D13-K)
- R13 pad 1: /VBATT_trig_manual -> Net-(D13-K)
- R7 pad 1: 5V0_GATED -> VBATT_GATED
- U1 pad 17: unconnected-(U1-P0.6-Pad17) -> /Batt_Low_Flag
- U1 pad 6: /Batt_Low_Flag -> unconnected-(U1-P1.7-Pad6)
- U6 pad 26: unconnected-(U6-GPIO45-Pad26) -> /ESPIO45
- U7 pad 5: GND -> /5V_EN
Routing:
- net Net-(D13-K): track 0.00 -> 40.5 mm, vias 0 -> 2
- net /VBATT_trig_manual: track 44.2 -> 4.35 mm, vias 2 -> 0
- net /ESPIO48: track 31.5 -> 7.79 mm, vias 1 -> 0
- net /Batt_Low_Flag: track 140.8 -> 119.3 mm, vias 5 -> 4
- net +3V3: track 91.4 -> 110.8 mm
- net /ESPIO47: track 26.1 -> 7.11 mm, vias 1 -> 0
- net /5V_EN: track 0.00 -> 18.4 mm
- net Net-(U5-VBUS): track 31.4 -> 17.3 mm, vias 2 -> 0
- net /ESPIO45: track 0.00 -> 13.6 mm, vias 0 -> 2
- net 5V0_GATED: track 31.3 -> 40.7 mm
- net GND: track 0.11 -> 7.57 mm, vias 363 -> 427
- net /ESP32_Module/DTR: track 33.8 -> 40.4 mm
- net Net-(Q4-B): track 6.24 -> 1.73 mm
- net /SCL: track 71.7 -> 68.0 mm
- net /ESPIO12: track 18.8 -> 22.0 mm
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Other:
- board text added: "POWER ON"
- board text added: "Pippino II board v2.1 May 2023"
- board text added: "Pippino II board v2.1 Pajaz design May 2023"
- board text removed: "5V GATED"
- board text removed: "PWR"
- board text removed: "Pippino II board v2.1 Apr 2023"
- board text removed: "Pippino II board v2.1 Pajaz design Apr 2023"
- board text removed: "START"
