File: Projects/Pippino_board_brushless_v2.1/pippino_board/pippino_board.kicad_sch (KiCad schematic)
At the start: 32 parts, among them J1 Conn_02x06_Odd_Even, J11 Conn_02x01, J2 Conn_02x01, J3 Conn_02x06_Odd_Even, J4 Conn_02x02_Counter_Clockwise, J5 Conn_02x09_Odd_Even, J6 Conn_02x03, J7 Conn_02x03, J8 Conn_02x02_Odd_Even, SW1 SW_Push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

Commit message: work on pippino II board v2.1
Other:
- title: (none) -> Pippino II Schematic v2.1
Changed lines of the file:
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@@
 (kicad_sch (version 20230121) (generator eeschema)
   (paper "A4")
+  (title_block
+    (title "Pippino II Schematic v2.1")
+  )
   (junction (at 64.77 104.14) (diameter 0) (color 0 0 0 0)
   )

Commit message: changed 5v buck to smaller one
Parts:
- added TP1: 5V_EN, TestPoint:TestPoint_Loop_D1.80mm_Drill1.0mm_Beaded, symbol Connector:TestPoint_Probe
Connections:
- new net 5V_EN: TP1.1
Other:
- sheet PSU_Gated ports: added 5V_EN; removed none
Changed lines of the file:
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@@
+    (stroke (width 0) (type default))
+  )
+  (wire (pts (xy 115.57 156.21) (xy 129.54 156.21))
     (stroke (width 0) (type default))
   )
@@
   )
   (label "Batt_Low_Flag" (at 77.47 128.27 0) (fields_autoplaced)
+    (effects (font (size 1.27 1.27)) (justify left bottom))
+  )
+  (label "5V_EN" (at 115.57 156.21 0) (fields_autoplaced)
     (effects (font (size 1.27 1.27)) (justify left bottom))
   )
@@
         (path "/dedb2da3-2254-430c-8837-0c4d082ac264"
           (reference "C2") (unit 1)
+        )
+      )
+    )
+  )
+  (symbol (lib_id "Connector:TestPoint_Probe") (at 115.57 156.21 180) (unit 1)
+    (in_bom yes) (on_board yes) (dnp no) (fields_autoplaced)
+    (property "Reference" "TP1" (at 116.84 157.1625 0)
+      (effects (font (size 1.27 1.27)) (justify right))
+    )
+    (property "Value" "5V_EN" (at 116.84 159.7025 0)
+      (effects (font (size 1.27 1.27)) (justify right))
+    )
+    (property "Footprint" "TestPoint:TestPoint_Loop_D1.80mm_Drill1.0mm_Beaded" (at 110.49 156.21 0)
+      (effects (font (size 1.27 1.27)) hide)
+    )
+    (property "Datasheet" "~" (at 110.49 156.21 0)
+      (effects (font (size 1.27 1.27)) hide)
+    )
+    (pin "1")
+    (instances
+      (project "pippino_board"
+        (path "/dedb2da3-2254-430c-8837-0c4d082ac264"
+          (reference "TP1") (unit 1)
         )
       )
@@
       (effects (font (size 1.27 1.27)) (justify right))
     )
-    (instances
+    (pin "5V_EN" input (at 129.54 156.21 180)
+      (effects (font (size 1.27 1.27)) (justify left))
+    )
+    (instances

Commit message: moved to ubu 22, updated pippino v2.1
Parts:
- added J12: Conn_02x02_Odd_Even, Connector_PinHeader_2.54mm:PinHeader_2x02_P2.54mm_Vertical, symbol Connector_Generic:Conn_02x02_Odd_Even
- added JP3: SolderJumper_2_Open, Jumper:SolderJumper-2_P1.3mm_Open_RoundedPad1.0x1.5mm, symbol Jumper:SolderJumper_2_Open
- added TP3: VB, TestPoint:TestPoint_Pad_D1.5mm, symbol Connector:TestPoint_Probe
- J1: footprint Connector_PinHeader_2.54mm:PinHeader_2x07_P2.54mm_Vertical -> Connector_PinHeader_2.54mm:PinHeader_2x08_P2.54mm_Vertical; symbol Connector_Generic:Conn_02x07_Odd_Even -> Connector_Generic:Conn_02x08_Odd_Even
- J5: value Conn_02x09_Odd_Even -> Conn_02x08_Odd_Even; footprint Connector_PinHeader_2.54mm:PinHeader_2x09_P2.54mm_Vertical -> Connector_PinHeader_2.54mm:PinHeader_2x08_P2.54mm_Vertical; symbol Connector_Generic:Conn_02x09_Odd_Even -> Connector_Generic:Conn_02x08_Odd_Even
- R7: value 330 -> 1K
- R8: value 18k -> 18K
- R9: value 5.1k -> 5.1K
- TP1: value 5V_EN -> VBG; footprint TestPoint:TestPoint_Loop_D1.80mm_Drill1.0mm_Beaded -> TestPoint:TestPoint_Pad_D1.5mm
Connections:
- net +3V3: now also J1.4 (Pin_4)
- net +BATT: now also TP3.1
- net 5V0_GATED: no longer J11.2 (Pin_2), R7.1
- net 5V_EN: now also JP3.2 (B); no longer TP1.1
- net Batt_Low_Flag: now also U1.17 (P0.6); no longer U1.6 (P1.7)
- net E18DC: now also J1.6 (Pin_6); no longer J1.4 (Pin_4)
- net E18DD: now also J1.8 (Pin_8); no longer J1.6 (Pin_6)
- net E18P14: now also J1.7 (Pin_7); no longer J1.5 (Pin_5)
- net E18P15: now also J1.9 (Pin_9); no longer J1.7 (Pin_7)
- net E18P16: now also J1.10 (Pin_10); no longer J1.8 (Pin_8)
- net E18RST: now also J1.5 (Pin_5); no longer J1.3 (Pin_3)
- net E18RX: now also J1.11 (Pin_11); no longer J1.9 (Pin_9)
- net E18TX: now also J1.12 (Pin_12); no longer J1.10 (Pin_10)
- net ESPIO12: now also J5.15 (Pin_15); no longer J5.17 (Pin_17)
- net ESPIO14: now also J5.16 (Pin_16); no longer J5.15 (Pin_15)
- net ESPIO47: now also J12.4 (Pin_4); no longer J5.18 (Pin_18)
- net ESPIO48: now also J12.3 (Pin_3); no longer J5.16 (Pin_16)
- net GND: now also J1.3 (Pin_3), J12.1 (Pin_1), J12.2 (Pin_2)
- net LED1: now also J1.16 (Pin_16); no longer J1.14 (Pin_14)
- net LED2: now also J1.15 (Pin_15); no longer J1.13 (Pin_13)
- net NWK_LED: now also J1.14 (Pin_14); no longer J1.12 (Pin_12)
- net RUN_LED: now also J1.13 (Pin_13); no longer J1.11 (Pin_11)
- net VBATT_GATED: now also J11.2 (Pin_2), R7.1, TP1.1
- new net ESPIO45: JP3.1 (A)
Other:
- sheet ESP32_Module ports: added GPIO45; removed none
- moved on the sheet: C1, D1, D2, R1, R2, R8, R9
